Commit message: Updated dependencies and added color for gazebo

File: urdf/description.gazebo.xacro (robot description, xacro)
@@ -1,6 +1,63 @@
 <?xml version="1.0"?>
+<!--
+Software License Agreement (BSD)
+\file      description.gazebo.xacro
+\authors   Raffaello Bonghi <raffaello.bonghi@officinerobotiche.it
+\copyright Copyright (c) 2015, Officine Robotiche, All rights reserved.
+Redistribution and use in source and binary forms, with or without modification, are permitted provided that
+the following conditions are met:
+ * Redistributions of source code must retain the above copyright notice, this list of conditions and the
+   following disclaimer.
+ * Redistributions in binary form must reproduce the above copyright notice, this list of conditions and the
+   following disclaimer in the documentation and/or other materials provided with the distribution.
+ * Neither the name of Clearpath Robotics nor the names of its contributors may be used to endorse or promote
+   products derived from this software without specific prior written permission.
+THIS SOFTWARE IS PROVIDED BY THE COPYRIGHT HOLDERS AND CONTRIBUTORS "AS IS" AND ANY EXPRESS OR IMPLIED WAR-
+RANTIES, INCLUDING, BUT NOT LIMITED TO, THE IMPLIED WARRANTIES OF MERCHANTABILITY AND FITNESS FOR A PARTICULAR
+PURPOSE ARE DISCLAIMED. IN NO EVENT SHALL THE COPYRIGHT HOLDER OR CONTRIBUTORS BE LIABLE FOR ANY DIRECT, IN-
+DIRECT, INCIDENTAL, SPECIAL, EXEMPLARY, OR CONSEQUENTIAL DAMAGES (INCLUDING, BUT NOT LIMITED TO, PROCUREMENT
+OF SUBSTITUTE GOODS OR SERVICES; LOSS OF USE, DATA, OR PROFITS; OR BUSINESS INTERRUPTION) HOWEVER CAUSED AND
+ON ANY THEORY OF LIABILITY, WHETHER IN CONTRACT, STRICT LIABILITY, OR TORT (INCLUDING NEGLIGENCE OR OTHERWISE)
+ARISING IN ANY WAY OUT OF THE USE OF THIS SOFTWARE, EVEN IF ADVISED OF THE POSSIBILITY OF SUCH DAMAGE.
+-->
 <robot name="dude_robot_gazebo" xmlns:xacro="http://ros.org/wiki/xacro">
   <xacro:include filename="$(find ros_dude_description)/urdf/dude.urdf.xacro" />
   <xacro:dude_robot />
+  <!-- base_link -->
+  <gazebo reference="base_link">
+    <material>Gazebo/Yellow</material>
+  </gazebo>
+  <!-- column_body_Link -->
+  <gazebo reference="column_body_Link">
+    <material>Gazebo/Black</material>
+  </gazebo>
+  <!-- electronics_Link -->
+  <gazebo reference="electronics_Link">
+    <material>Gazebo/Green</material>
+  </gazebo>
+  <!-- wall_body_Link -->
+  <!--<gazebo reference="wall_body_Link">
+    <material>Gazebo/WhiteEmissive</material>
+  </gazebo>-->
+  <!-- battery_Link -->
+  <gazebo reference="battery_Link">
+    <material>Gazebo/Black</material>
+  </gazebo>
+  <!-- Differential drive -->
+	<gazebo>
+		<plugin name="differential_drive_controller" filename="libgazebo_ros_diff_drive.so">
+		  <alwaysOn>true</alwaysOn>
+		  <updateRate>10.0</updateRate>
+		  <leftJoint>left</leftJoint>
+		  <rightJoint>right</rightJoint>
+		  <wheelSeparation>0.5380</wheelSeparation>
+		  <wheelDiameter>0.2410</wheelDiameter>
+		  <torque>20</torque>
+		  <commandTopic>cmd_vel</commandTopic>
+		  <odometryTopic>odom</odometryTopic>
+		  <odometryFrame>odom</odometryFrame>
+		  <robotBaseFrame>base_link</robotBaseFrame>
+		</plugin>
+	</gazebo>
   <!--<xacro:include filename="$(find ros_dude_description)/urdf/dude.urdf.xacro" />
   <xacro:include filename="$(find rodo_dude_gazebo)/urdf/dude.gazebo.xacro" />-->
@@ -11,5 +68,3 @@
     </plugin>
   </gazebo>-->
-  <!--<xacro:dude />-->
-  <!--<xacro:husky_robot_gazebo />-->
 </robot>

Commit message: Removed namespace

File: urdf/description.gazebo.xacro (robot description, xacro)
@@ -22,8 +22,7 @@
 -->
 <robot name="dude_robot_gazebo" xmlns:xacro="http://ros.org/wiki/xacro">
-  <xacro:arg name="robot_name" default="dude_gazebo" />
   <xacro:include filename="$(find ros_dude_gazebo)/urdf/xtion_camera.gazebo.xacro"/>
   <xacro:include filename="$(find ros_dude_description)/urdf/dude.urdf.xacro" />
-  <xacro:dude_robot />
+  <xacro:macro name="dude_robot_gazebo">
   <!-- base_link -->
   <gazebo reference="base_link">
@@ -46,5 +45,5 @@
     <material>Gazebo/Black</material>
   </gazebo>
-  <!--<xacro:xtion_camera_gazebo prefix="xtion_camera"/>-->
+  <xacro:xtion_camera_gazebo prefix="xtion_camera"/>
   <!-- Differential drive -->
 	<gazebo>
@@ -57,7 +56,7 @@
 		  <wheelDiameter>${wheel_radius*2}</wheelDiameter>
 		  <torque>20</torque>
-		  <commandTopic>/$(arg robot_name)/cmd_vel</commandTopic>
-		  <odometryTopic>/$(arg robot_name)/odom</odometryTopic>
-		  <odometryFrame>/$(arg robot_name)/odom</odometryFrame>
+		  <commandTopic>/cmd_vel</commandTopic>
+		  <odometryTopic>/odom</odometryTopic>
+		  <odometryFrame>/odom</odometryFrame>
 		  <robotBaseFrame>base_link</robotBaseFrame>
       <publishWheelTF>true</publishWheelTF>
@@ -71,3 +70,4 @@
     </plugin>
   </gazebo>-->
+</xacro:macro>
 </robot>

Commit message: Added ros_controller

File: urdf/description.gazebo.xacro (robot description, xacro)
@@ -24,5 +24,23 @@
   <xacro:include filename="$(find ros_dude_gazebo)/urdf/xtion_camera.gazebo.xacro"/>
   <xacro:include filename="$(find ros_dude_description)/urdf/dude.urdf.xacro" />
-  <xacro:macro name="dude_robot_gazebo">
+  <xacro:dude_robot_gazebo />
+  <!-- Differential drive -->
+	<gazebo>
+		<plugin name="differential_drive_controller" filename="libgazebo_ros_diff_drive.so">
+		  <alwaysOn>true</alwaysOn>
+		  <updateRate>10.0</updateRate>
+		  <leftJoint>left</leftJoint>
+		  <rightJoint>right</rightJoint>
+		  <wheelSeparation>${wheel_offset_y*2}</wheelSeparation>
+		  <wheelDiameter>${wheel_radius*2}</wheelDiameter>
+		  <torque>20</torque>
+		  <commandTopic>cmd_vel</commandTopic>
+		  <odometryTopic>odom</odometryTopic>
+		  <odometryFrame>odom</odometryFrame>
+		  <robotBaseFrame>base_link</robotBaseFrame>
+      <publishWheelTF>true</publishWheelTF>
+      <publishWheelJointState>true</publishWheelJointState>
+		</plugin>
+	</gazebo>
   <!-- base_link -->
   <gazebo reference="base_link">
@@ -46,28 +64,3 @@
   </gazebo>
   <xacro:xtion_camera_gazebo prefix="xtion_camera"/>
-  <!-- Differential drive -->
-	<gazebo>
-		<plugin name="differential_drive_controller" filename="libgazebo_ros_diff_drive.so">
-		  <alwaysOn>true</alwaysOn>
-		  <updateRate>10.0</updateRate>
-		  <leftJoint>right</leftJoint>
-		  <rightJoint>left</rightJoint>
-		  <wheelSeparation>${wheel_offset_y*2}</wheelSeparation>
-		  <wheelDiameter>${wheel_radius*2}</wheelDiameter>
-		  <torque>20</torque>
-		  <commandTopic>/cmd_vel</commandTopic>
-		  <odometryTopic>/odom</odometryTopic>
-		  <odometryFrame>/odom</odometryFrame>
-		  <robotBaseFrame>base_link</robotBaseFrame>
-      <publishWheelTF>true</publishWheelTF>
-      <publishWheelJointState>true</publishWheelJointState>
-		</plugin>
-	</gazebo>
-  <!-- Gazebo plugin for ROS Control -->
-  <!--<gazebo>
-    <plugin name="gazebo_ros_control" filename="libgazebo_ros_control.so">
-      <robotNamespace>/</robotNamespace>
-    </plugin>
-  </gazebo>-->
-</xacro:macro>
 </robot>

Commit message: Fixed information about camera and link

File: urdf/description.gazebo.xacro (robot description, xacro)
@@ -25,22 +25,4 @@
   <xacro:include filename="$(find ros_dude_description)/urdf/dude.urdf.xacro" />
   <xacro:dude_robot_gazebo />
-  <!-- Differential drive -->
-	<gazebo>
-		<plugin name="differential_drive_controller" filename="libgazebo_ros_diff_drive.so">
-		  <alwaysOn>true</alwaysOn>
-		  <updateRate>10.0</updateRate>
-		  <leftJoint>left</leftJoint>
-		  <rightJoint>right</rightJoint>
-		  <wheelSeparation>${wheel_offset_y*2}</wheelSeparation>
-		  <wheelDiameter>${wheel_radius*2}</wheelDiameter>
-		  <torque>20</torque>
-		  <commandTopic>cmd_vel</commandTopic>
-		  <odometryTopic>odom</odometryTopic>
-		  <odometryFrame>odom</odometryFrame>
-		  <robotBaseFrame>base_link</robotBaseFrame>
-      <publishWheelTF>true</publishWheelTF>
-      <publishWheelJointState>true</publishWheelJointState>
-		</plugin>
-	</gazebo>
   <!-- base_link -->
   <gazebo reference="base_link">
@@ -56,11 +38,29 @@
   </gazebo>
   <!-- wall_body_Link -->
-  <!--<gazebo reference="wall_body_Link">
-    <material>Gazebo/WhiteEmissive</material>
-  </gazebo>-->
+  <gazebo reference="wall_body_Link">
+    <material>Gazebo/White</material>
+  </gazebo>
   <!-- battery_Link -->
   <gazebo reference="battery_Link">
-    <material>Gazebo/Black</material>
+    <material>Gazebo/Blue</material>
   </gazebo>
-  <xacro:xtion_camera_gazebo prefix="xtion_camera"/>
+  <!--<xacro:xtion_camera_gazebo prefix="xtion_camera"/>-->
+  <!-- Differential drive -->
+	<gazebo>
+		<plugin name="differential_drive_controller" filename="libgazebo_ros_diff_drive.so">
+		  <alwaysOn>true</alwaysOn>
+		  <updateRate>10.0</updateRate>
+		  <leftJoint>Left</leftJoint>
+		  <rightJoint>Right</rightJoint>
+		  <wheelSeparation>${wheel_offset_y*2}</wheelSeparation>
+		  <wheelDiameter>${wheel_radius*2}</wheelDiameter>
+		  <torque>20</torque>
+		  <commandTopic>cmd_vel</commandTopic>
+		  <odometryTopic>odom</odometryTopic>
+		  <odometryFrame>odom</odometryFrame>
+		  <robotBaseFrame>base_link</robotBaseFrame>
+      <publishWheelTF>true</publishWheelTF>
+      <publishWheelJointState>true</publishWheelJointState>
+		</plugin>
+	</gazebo>
 </robot>

File: urdf/xtion_camera.gazebo.xacro (robot description, xacro)
@@ -2,16 +2,16 @@
 <root xmlns:xacro="http://ros.org/wiki/xacro">
 <xacro:macro name="xtion_camera_gazebo" params="prefix">
-  <joint name="${prefix}_optical_joint" type="fixed">
+  <joint name="${prefix}_joint_optical" type="fixed">
     <origin xyz="0 0 0" rpy="-1.5708 0 -1.5708"/>
     <parent link="${prefix}_Link"/>
-    <child link="${prefix}_frame_optical"/>
+    <child link="${prefix}_optical_frame"/>
   </joint>
-  <link name="${prefix}_frame_optical"/>
-  <gazebo reference="${prefix}_Link">
-    <sensor type="depth" name="${prefix}">
+  <link name="${prefix}_optical_frame"/>
+  <gazebo reference="camera_rgb_frame">
+    <sensor type="depth" name="xtion_camera">
       <always_on>true</always_on>
       <update_rate>20.0</update_rate>
       <camera>
-        <horizontal_fov>${60.0*M_PI/180.0}</horizontal_fov>
+        <horizontal_fov>${58.0*M_PI/180.0}</horizontal_fov>
         <image>
           <format>R8G8B8</format>
@@ -20,10 +20,10 @@
         </image>
         <clip>
-          <near>0.05</near>
-          <far>8.0</far>
+          <near>0.08</near>
+          <far>3.0</far>
         </clip>
       </camera>
-      <plugin name="kinect_${prefix}_controller" filename="libgazebo_ros_openni_kinect.so">
-        <cameraName>${prefix}</cameraName>
+      <plugin name="xtion_camera_controller" filename="libgazebo_ros_openni_kinect.so">
+        <cameraName>xtion_camera</cameraName>
         <alwaysOn>true</alwaysOn>
         <updateRate>10</updateRate>
@@ -33,5 +33,5 @@
         <cameraInfoTopicName>rgb/camera_info</cameraInfoTopicName>
         <depthImageCameraInfoTopicName>depth/camera_info</depthImageCameraInfoTopicName>
-        <frameName>${prefix}_frame_optical</frameName>
+        <frameName>camera_rgb_optical_frame</frameName>
         <baseline>0.1</baseline>
         <distortion_k1>0.0</distortion_k1>
